File: hardware/PCB/TopiaryTrimbot.kicad_pcb (KiCad board)
At the start: 2 copper layers, 284 parts, among them J1 24V LED Strip, J10 Conn_01x03, J11 Conn_01x03, J12 USB_C_Receptacle_USB2.0_16P, J13 Conn_02x05_Odd_Even, J14 Turntable Stepper, J15 Gantry Stepper, J16 Extruder Stepper, J17 Revolute Stepper, J18 Cutting Tool, J19 Conn_01x03, J2 24V FAN XYJ24B4010M, J20 Conn_02x20_Odd_Even, J21 MEM2052-00-195-00-A, J3 Power Entry, J4 Conn_01x03, J5 Conn_01x03, J6 Conn_01x03, J7 Conn_01x03, J8 Conn_01x03, J9 Conn_01x03, SW1 RESET, SW2 PROG, U1 TPS62933, U10 BSC050N04LSG, U11 EMIF06-MSD02N16, U12 MT25QL128ABA1ESE-0SIT, U13 TPS923650, U14 TSC2013QRSARQ1, U2 XL4015 Regulator Module, U3 XL4015 Regulator Module, U4 TPS56837Hx, U5 XL4015 Regulator Module, U6 TPS56837Hx, U7 32 MHz, U8 STM32H747IITx, U9 USBLC6-2, Y1 Crystal

Commit message: Finish first pass placement of parts on PCB, several updates and fixes to schematic included
Parts:
- removed the C44 at (264.5, 145.3)
- removed the C45 at (271.9, 107.1)
- removed the R15 at (243.4, 135.5)
- removed the R16 at (243.4, 138.4)
- removed the R19 at (243.4, 147.3)
- removed the R20 at (243.4, 150.2)
- removed the R21 at (247.9, 135.5)
- removed the R22 at (247.9, 138.4)
- removed the U4 at (205.9, 81.3)
- removed the U6 at (205.9, 85.7)
- added C57: 4.7u, Capacitor_SMD:C_0805_2012Metric, B.Cu at (324.6, 134.6)
- added C58: 1u, Capacitor_SMD:C_0805_2012Metric, F.Cu at (345.5, 107.5)
- added C59: 1u, Capacitor_SMD:C_0805_2012Metric, F.Cu at (334.1, 107.5)
- added C60: 1u, Capacitor_SMD:C_0805_2012Metric, F.Cu at (322.6, 107.5)
- added C61: 1u, Capacitor_SMD:C_0805_2012Metric, F.Cu at (311.2, 107.5)
- added C62: 1u, Capacitor_SMD:C_0805_2012Metric, F.Cu at (299.8, 107.5)
- added C63: 1u, Capacitor_SMD:C_0805_2012Metric, F.Cu at (355.2, 163.3)
- added R24: 4.7k, Resistor_SMD:R_0805_2012Metric, F.Cu at (330.3, 170.9)
- added R25: 4.7k, Resistor_SMD:R_0805_2012Metric, F.Cu at (333.1, 170.9)
- added U2: TPS56837Hx, CustomFootprints:RPA0010A-MFG, F.Cu at (246.9, 150.6)
- added U3: TPS56837Hx, CustomFootprints:RPA0010A-MFG, F.Cu at (246.8, 181.0)
- C30: renamed from C28; moved to B.Cu
- C32: renamed from C50; moved to B.Cu
- C35: renamed from C29; moved to B.Cu
- C36: renamed from C47; moved to B.Cu
- C37: renamed from C30; moved to B.Cu
- C38: renamed from C51; moved to B.Cu
- C39: renamed from C31; moved to B.Cu
- C40: renamed from C32; moved to B.Cu
- C41: renamed from C33; moved to B.Cu
- C42: renamed from C48; moved to B.Cu
- C43: renamed from C34; moved to B.Cu
- C44: renamed from C35; moved to B.Cu
- C45: renamed from C52; moved to B.Cu
- C46: renamed from C36; moved to B.Cu
- C47: renamed from C37; moved to B.Cu
- C48: renamed from C53; moved to B.Cu
- C49, TP21, TP22, TP23, TP24, TP25, TP26, U12: moved to B.Cu
- C50: renamed from C38; moved to B.Cu
- C51: renamed from C39; moved to B.Cu
- C52: renamed from C40; moved to B.Cu
- C53: renamed from C41; moved to B.Cu
- C54: renamed from C42; moved to B.Cu
- C55: renamed from C43; moved to B.Cu
- C69: renamed from C63; moved to B.Cu
- DS1: footprint Connector_FFC-FPC:Hirose_FH12-40S-0.5SH_1x40-1MP_P0.50mm_Horizontal -> CustomFootprints:Hirose_FH12A-40S-0.5SH_1x40-1MP_P0.50mm_Horizontal
- JP1, JP2, JP3: footprint Jumper:SolderJumper-3_P2.0mm_Open_TrianglePad1.0x1.5mm -> CustomFootprints:SolderJumper-3_P1.5mm_Open_RoundedPad1.0x1.5mm
- R13: renamed from R10; value 1.3k -> 1k
- R26: renamed from R28; moved to B.Cu
- R27: renamed from R29; moved to B.Cu
- R38: renamed from R42; moved to B.Cu
- moved R50 228.2 mm to (367.1, 197.6), turned to -90 degrees
- moved R51 226.8 mm to (365.6, 197.6), turned to -90 degrees
- moved R52 224.7 mm to (364.1, 197.6), turned to -90 degrees
- moved R53 222.6 mm to (362.6, 197.6), turned to -90 degrees
- moved R54 220.6 mm to (361.0, 197.6), turned to -90 degrees
- moved R55 218.0 mm to (359.5, 197.6), turned to -90 degrees
- moved R56 216.1 mm to (358.0, 197.6), turned to -90 degrees
- moved R57 213.7 mm to (356.5, 197.6), turned to -90 degrees
- moved R58 212.6 mm to (354.9, 197.6), turned to -90 degrees
- moved H4 211.2 mm to (380.0, 80.0)
- moved R59 210.4 mm to (353.4, 197.6), turned to -90 degrees
- moved R60 208.3 mm to (351.9, 197.6), turned to -90 degrees
- moved R61 206.3 mm to (350.4, 197.6), turned to -90 degrees
- moved R62 203.7 mm to (348.8, 197.6), turned to -90 degrees
- moved R63 201.7 mm to (347.3, 197.6), turned to -90 degrees
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- renumbered A3 to A2, A2 to A3, C20 to C11, C3 to C12, C15 to C13, C25 to C14, C16 to C15, C26 to C16, C5 to C17, C6 to C18, C11 to C19, C8 to C2, C21 to C20, C7 to C21, C12 to C22, C22 to C23, C13 to C24, C23 to C25, C14 to C26, C24 to C27, C54 to C28, C55 to C29, C18 to C3, C46 to C31, C56 to C33, C57 to C34, C17 to C4, C27 to C5, C2 to C6, C58 to C65, C60 to C66, C59 to C67, C61 to C68, C9 to C7, C62 to C70, C64 to C71, C70 to C72, C65 to C73, C66 to C74, C73 to C75, C71 to C76, C74 to C77, C75 to C78, C72 to C79, C19 to C8, C67 to C80, C68 to C81, C69 to C82, C4 to C9, D3 to D1, D14 to D13, D13 to D14, D6 to D2, D1 to D3, D2 to D4, D4 to D6, J11 to J10, J12 to J11, J7 to J12, J9 to J13, J16 to J15, J18 to J16, J15 to J17, J17 to J18, J20 to J19, J19 to J20, J13 to J4, J4 to J5, J5 to J6, J6 to J7, J10 to J9, JP14 to JP10, JP18 to JP11, JP20 to JP12, JP22 to JP13, JP5 to JP14, JP17 to JP15, JP7 to JP16, JP9 to JP17, JP11 to JP18, JP13 to JP19, JP15 to JP20, JP19 to JP21, JP21 to JP22, JP26 to JP24, JP24 to JP25, JP25 to JP26, JP16 to JP5, JP8 to JP7, JP10 to JP8, JP12 to JP9, R8 to R1, R11 to R10, R1 to R11, R4 to R12, R9 to R14, R27 to R15, R30 to R16, R23 to R17, R24 to R18, R25 to R19, R14 to R2, R26 to R20, R17 to R21, R18 to R22, R31 to R23, R32 to R28, R36 to R29, R6 to R3, R34 to R30, R38 to R31, R40 to R32, R41 to R33, R33 to R34, R37 to R35, R35 to R36, R39 to R37, R76 to R39, R12 to R4, R77 to R40, R54 to R41, R78 to R42, R60 to R43, R79 to R44, R51 to R45, R82 to R46, R44 to R47, R46 to R48, R43 to R49, R2 to R5, R45 to R50, R47 to R51, R48 to R52, R49 to R53, R50 to R54, R52 to R55, R53 to R56, R55 to R57, R56 to R58, R57 to R59, R3 to R6, R58 to R60, R59 to R61, R61 to R62, R62 to R63, R63 to R64, R64 to R65, R65 to R66, R66 to R67, R67 to R68, R68 to R69, R13 to R7, R69 to R70, R70 to R71, R71 to R72, R72 to R73, R73 to R74, R74 to R75, R75 to R76, R80 to R77, R81 to R78, R5 to R8, R7 to R9, TP7 to TP10, TP9 to TP11, TP11 to TP12, TP8 to TP7, TP10 to TP8, TP12 to TP9, U2 to U4, U3 to U5, U5 to U6
Connections:
- A2 pad 3: Net-(A3-A2) -> Net-(A2-A2)
- A2 pad 4: Net-(A3-A1) -> Net-(A2-A1)
- A3 pad 3: Net-(A2-A2) -> Net-(A3-A2)
- A3 pad 4: Net-(A2-A1) -> Net-(A3-A1)
- D11 pad 1: VBUS -> Net-(D11-K)
- J11 pad A4: Net-(D11-A) -> VBUS
- J11 pad A9: Net-(D11-A) -> VBUS
- J11 pad B4: Net-(D11-A) -> VBUS
- J11 pad B9: Net-(D11-A) -> VBUS
- J12 pad 1: /MCU/AUX_SCL -> /MCU/UART6_TX
- J12 pad 2: /MCU/AUX_SDA -> /MCU/UART6_RX
- J13 pad 1: /MCU/UART6_TX -> /MCU/AUX_SCL
- J13 pad 2: /MCU/UART6_RX -> /MCU/AUX_SDA
- J14 pad 1: Net-(A1-A1) -> Net-(A1-A2)
- J14 pad 2: Net-(A1-A2) -> Net-(A1-A1)
- J15 pad 1: Net-(A3-A1) -> Net-(A2-A2)
- J15 pad 2: Net-(A3-A2) -> Net-(A2-A1)
- J17 pad 1: Net-(A2-A1) -> Net-(A3-A2)
- J17 pad 2: Net-(A2-A2) -> Net-(A3-A1)
- J18 pad 1: Net-(A4-A1) -> Net-(A4-A2)
- J18 pad 2: Net-(A4-A2) -> Net-(A4-A1)
- R21 pad 2: Net-(U8-PA9) -> Net-(D11-A)
- R22 pad 1: Net-(U8-PA9) -> Net-(D11-A)
- U8 pad 128: Net-(U8-PA9) -> Net-(D11-K)
- U8 pad 132: unconnected-(U8-PA13-Pad132) -> /MCU/SWDIO
- U8 pad 138: unconnected-(U8-PA14-Pad138) -> /MCU/SWCLK
- U9 pad 1: /MCU/USB_DM -> /MCU/USB_DP
- U9 pad 3: /MCU/USB_DP -> /MCU/USB_DM
- U9 pad 4: /MCU/USB_DP -> /MCU/USB_DM
- U9 pad 6: /MCU/USB_DM -> /MCU/USB_DP
Routing:
- net (no net): vias 0 -> 4
Other:
- board outline added: 190.5 x 160 mm
- copper layers 2 -> 4
- board text added: "+ 24VDC in -"
- board text added: "+ Cutter -"
- board text added: "-Fan+"
- board text added: "-LED+"
- board text added: "24V Status"
- board text added: "3.3V Status"
- board text added: "5-15V Fault"
- board text added: "5-15V Status"
- board text added: "5V Fault"
- board text added: "5V Status"
- board text added: "An ECE49595 Project by"
- board text added: "Bypass"
- board text added: "Door SW"
- board text added: "Extruder"
- board text added: "Extruder SW"
- board text added: "GND"
- board text added: "Gantry"
- board text added: "Gantry SW"
- board text added: "Griffin Ross, Thomas Schorer Jackson Duke, and Collin Shanks"
- board text added: "LCD"
- board text added: "Program"
- board text added: "Reset"
- board text added: "Revolute"
- board text added: "Revolute SW"
- board text added: "TX RX GND"
- board text added: "Topiary Trimbot"
- board text added: "Turntable"
- board text added: "Turntable SW"
