File: hardware/PCB/TopiaryTrimbot.kicad_pcb (KiCad board)
At the start: 4 copper layers, 190.5 x 160 mm, 285 parts, among them J1 24V LED Strip, J10 Conn_01x03, J11 USB_C_Receptacle_USB2.0_16P, J12 Conn_01x03, J13 Conn_01x03, J14 Turntable Stepper, J15 Extruder Stepper, J16 Cutting Tool, J17 Gantry Stepper, J18 Revolute Stepper, J19 Conn_02x20_Odd_Even, J2 24V FAN XYJ24B4010M, J20 Conn_01x03, J21 MEM2090-00-145-00-A, J3 Power Entry, J4 Conn_02x05_Odd_Even, J5 Conn_01x03, J6 Conn_01x03, J7 Conn_01x03, J8 Conn_01x03, J9 Conn_01x03, SW1 RESET, SW2 PROG, U1 TPS62933, U10 BSC050N04LSG, U11 EMIF06-MSD02N16, U12 MX25L51245GZ2I-08G, U13 STCS2ASPR, U14 TSC2013QRSARQ1, U2 TPS56837Hx, U3 TPS56837Hx, U4 XL4015 Regulator Module, U5 XL4015 Regulator Module, U6 XL4015 Regulator Module, U7 32 MHz, U8 STM32H747IITx, U9 USBLC6-2, Y1 Crystal

Commit message: Final PCB version sent for order
Parts:
- C71, R44, U12: moved to F.Cu
- moved R44 35.9 mm to (302.8, 146.3), turned to 180 degrees
- moved U12 27.6 mm to (307.2, 150.7), turned to 0 degrees
- moved C69 26.8 mm to (307.3, 150.9), turned to 180 degrees
- moved C34 14.4 mm to (296.9, 139.7), turned to 90 degrees
- moved R22 11.2 mm to (299.2, 139.7), turned to 90 degrees
- moved R21 10.5 mm to (300.2, 160.8)
- moved U7 6.79 mm to (309.5, 157.0)
- moved C37 6.72 mm to (309.5, 156.7)
- moved C16 6.29 mm to (246.6, 157.7)
- moved C33 5.40 mm to (296.7, 160.8)
- moved SW1 5.16 mm to (296.9, 155.4)
- moved SW2 5.15 mm to (296.9, 145.5)
- moved R10 5.02 mm to (250.2, 158.0), turned to 0 degrees
- moved C26 2.95 mm to (272.5, 182.1)
- moved C27 2.24 mm to (273.1, 151.5)
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Routing:
- net NOR_CS: track 11.1 -> 54.9 mm, vias 1 -> 4
- net /MCU/RESET: track 123.2 -> 133.7 mm, vias 5 -> 3
- net /MCU/OSC_IN: track 4.56 -> 11.9 mm
- net Net-(C16-Pad1): track 30.7 -> 37.3 mm
- net EXTRUDER_FLT: track 119.6 -> 113.7 mm
- net GND: track 155.6 -> 149.9 mm, vias 228 -> 442
- net PG_ADJ: track 100.2 -> 105.9 mm
- net Net-(U3-FB): track 13.7 -> 9.05 mm
- net TS_NRST: track 76.8 -> 81.2 mm, vias 0 -> 2
- net TURNTABLE_STEP: track 87.8 -> 83.5 mm, vias 4 -> 2
- net +3.3V: track 147.7 -> 143.4 mm, vias 43 -> 49
- net TS_INT: track 71.3 -> 75.6 mm, vias 0 -> 2
- net REVOLUTE_FLT: track 145.9 -> 141.7 mm
- net GANTRY_FLT: track 98.6 -> 94.6 mm
- net GANTRY_STEP: track 110.2 -> 106.5 mm, vias 4 -> 2
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