File: hardware/PCB/mcu.kicad_sch (KiCad schematic)
At the start: 73 parts, among them J10 Conn_01x03, J11 Conn_01x03, J12 USB_C_Receptacle_USB2.0_16P, J13 Conn_01x03, J2 Conn_02x05_Odd_Even, J5 Conn_01x03, J6 Conn_01x03, J7 Conn_01x03, J8 Conn_01x03, J9 Conn_01x03, SW1 RESET, SW2 PROG, U4 32 MHz, U5 USBLC6-2, Y1 Crystal

Commit message: Synchronized schematic draft and reannotated all
Parts:
- C54: renamed from C30; now not fitted
- C55: renamed from C31; now not fitted
- Y1: now not fitted
- gave numbers to parts that had none: 1
- renumbered C11 to C28, C10 to C29, C12 to C30, C13 to C31, C14 to C32, C15 to C33, C16 to C34, C17 to C35, C18 to C36, C19 to C37, C20 to C38, C21 to C39, C22 to C40, C23 to C41, C24 to C42, C25 to C43, C26 to C44, C9 to C45, C43 to C46, C46 to C47, C51 to C48, C27 to C49, C49 to C50, C50 to C51, C8 to C52, C7 to C53, C5 to C56, C6 to C57, D5 to D10, D6 to D11, D2 to D7, D3 to D8, D4 to D9, J9 to J10, J10 to J11, J2 to J13, J11 to J4, J13 to J7, J7 to J8, J8 to J9, R20 to R15, R21 to R16, R53 to R17, R56 to R18, R22 to R19, R23 to R20, R24 to R21, R25 to R22, R59 to R23, R60 to R24, R61 to R25, R62 to R26, R57 to R27, R55 to R28, R54 to R29, R58 to R30, R63 to R31, TP31 to TP1, TP26 to TP2, TP27 to TP3, TP28 to TP4, TP29 to TP5, U4 to U7, U5 to U9
Other:
- note added: "Debugging UART"
- note added: "Endstop Switches"
- note added: "Spare I2C"
- note added: "To POWER"
- moved on the sheet: J10, J11, J4, J5, J6, J7, J8, R15, R16, R19, R20, R21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

Commit message: Finish first pass placement of parts on PCB, several updates and fixes to schematic included
Parts:
- removed C44: 100n, Capacitor_SMD:C_0603_1608Metric, symbol Device:C
- removed C45: 4.7u, Capacitor_SMD:C_0805_2012Metric, symbol Device:C
- removed R15, R16, R19, R20, R21, R22: 10k, Resistor_SMD:R_0805_2012Metric, symbol Device:R_US
- added C57: 4.7u, Capacitor_SMD:C_0805_2012Metric, symbol Device:C
- added C58, C59, C60, C61, C62, C63: 1u, Capacitor_SMD:C_0805_2012Metric, symbol Device:C
- added R24, R25: 4.7k, Resistor_SMD:R_0805_2012Metric, symbol Device:R_US
- renumbered C54 to C28, C55 to C29, C28 to C30, C46 to C31, C50 to C32, C56 to C33, C57 to C34, C29 to C35, C47 to C36, C30 to C37, C51 to C38, C31 to C39, C32 to C40, C33 to C41, C48 to C42, C34 to C43, C35 to C44, C52 to C45, C36 to C46, C37 to C47, C53 to C48, C38 to C50, C39 to C51, C40 to C52, C41 to C53, C42 to C54, C43 to C55, J11 to J10, J12 to J11, J7 to J12, J9 to J13, J13 to J4, J4 to J5, J5 to J6, J6 to J7, J10 to J9, R27 to R15, R30 to R16, R23 to R17, R24 to R18, R25 to R19, R26 to R20, R17 to R21, R18 to R22, R31 to R23, R28 to R26, R29 to R27
Connections:
- net +3.3V: now also C57.1, R24.1, R25.1
- net AUX_SCL: now also J13.1 (Pin_1), R24.2; no longer J12.1 (Pin_1)
- net AUX_SDA: now also J13.2 (Pin_2), R25.2; no longer J12.2 (Pin_2)
- net AUX_SW: now also C63.1
- net DOOR_SW: now also C62.1
- net EXTRUDER_SW: now also C60.1
- net GANTRY_SW: now also C59.1
- net GND: now also C57.2, C58.2, C59.2, C60.2, C61.2, C62.2, C63.2
- net REVOLUTE_SW: now also C61.1
- net SWCLK: now also U8.138 (PA14)
- net SWDIO: now also U8.132 (PA13)
- net TURNTABLE_SW: now also C58.1
- net UART6_RX: now also J12.2 (Pin_2); no longer J13.2 (Pin_2)
- net UART6_TX: now also J12.1 (Pin_1); no longer J13.1 (Pin_1)
- net USB_DM: now also U9.3 (I/O2), U9.4 (I/O2); no longer U9.1 (I/O1), U9.6 (I/O1)
- net USB_DP: now also U9.1 (I/O1), U9.6 (I/O1); no longer U9.3 (I/O2), U9.4 (I/O2)
- net VBUS: now also J11.A4 (VBUS), J11.A9 (VBUS), J11.B4 (VBUS), J11.B9 (VBUS); no longer D11.1 (K)
- net at R21.2, R22.1: now also D11.2 (A); no longer U8.128 (PA9)
- new net: D11.1 (K), U8.128 (PA9)
- no-connect marks 46 -> 44
Other:
- moved on the sheet: D11, J13, R21, R22

Commit message: Started routing
Parts:
- added C37: 100n, Capacitor_SMD:C_0603_1608Metric, symbol Device:C
- added C48: 2.2u, Capacitor_SMD:C_0805_2012Metric, symbol Device:C
- renumbered C37 to C38, C38 to C39, C39 to C40, C40 to C41, C41 to C42, C42 to C43, C43 to C44, C44 to C45, C45 to C46, C46 to C47, C47 to C49, C48 to C50, C49 to C51, C50 to C52, C51 to C53, C52 to C54, C53 to C55, C54 to C56, C55 to C57, C57 to C58, C58 to C59, C59 to C60, C60 to C61, C61 to C62, C62 to C63, C63 to C64
Connections:
- net +3.3V: now also C37.1
- net GND: now also C37.2, C48.2
- net LCD_DE: now also U8.75 (PE13); no longer U8.30 (PF10)
- net NOR_CLK: now also U8.30 (PF10); no longer U8.57 (PB2)
- net NOR_D2: now also U8.27 (PF7); no longer U8.1 (PE2)
- net REVOLUTE_DIR: now also U8.110 (PG2); no longer U8.115 (PG5)
- net REVOLUTE_STEP: now also U8.95 (PD12); no longer U8.98 (PD15)
- net TS_INT: now also U8.21 (PF3); no longer U8.20 (PF2)
- net TS_NRST: now also U8.20 (PF2); no longer U8.22 (PF4)
- net TURNTABLE_DIR: now also U8.115 (PG5); no longer U8.110 (PG2)
- net TURNTABLE_STEP: now also U8.98 (PD15); no longer U8.95 (PD12)
- net VCAPDSI: now also C48.1
Other:
- note added: "DSI Decoupling"
- note removed: "need decoupling cap"
