File: hardware/PCB/mcu.kicad_sch (KiCad schematic)
At the start: 76 parts, among them J10 Conn_01x03, J11 USB_C_Receptacle_USB2.0_16P, J12 Conn_01x03, J13 Conn_01x03, J4 Conn_02x05_Odd_Even, J5 Conn_01x03, J6 Conn_01x03, J7 Conn_01x03, J8 Conn_01x03, J9 Conn_01x03, SW1 RESET, SW2 PROG, U7 32 MHz, U8 STM32H747IITx, U9 USBLC6-2, Y1 Crystal

Commit message: Continue layout, including swapping to linear BL driver
Parts:
- renumbered D8 to D10, D7 to D11, D11 to D7, D10 to D8, R15 to R21, R16 to R22, R21 to R23, R22 to R24, R20 to R25, R19 to R26, R18 to R27, R17 to R28, R23 to R29, R24 to R30, R25 to R31, R26 to R32, R27 to R33
Connections:
- net AUX_SW: now also U8.89 (PD8); no longer U8.85 (PB12)
- net CUTTER_EN: now also U8.35 (PC1); no longer U8.66 (PG1)
- net DOOR_SW: now also U8.162 (PB3); no longer U8.166 (PB7)
- net EXTRUDER_DIR: now also U8.165 (PB6); no longer U8.111 (PG3)
- net EXTRUDER_FLT: now also U8.22 (PF4); no longer U8.68 (PE8)
- net EXTRUDER_SW: now also U8.156 (PG12); no longer U8.164 (PB5)
- net GANTRY_DIR: now also U8.164 (PB5); no longer U8.114 (PG4)
- net GANTRY_FLT: now also U8.2 (PE3); no longer U8.69 (PE9)
- net GANTRY_SW: now also U8.155 (PG11); no longer U8.163 (PB4)
- net REVOLUTE_DIR: now also U8.166 (PB7); no longer U8.110 (PG2)
- net REVOLUTE_FLT: now also U8.23 (PF5); no longer U8.72 (PE10)
- net REVOLUTE_SW: now also U8.161 (PG15); no longer U8.165 (PB6)
- net TURNTABLE_DIR: now also U8.163 (PB4); no longer U8.115 (PG5)
- net TURNTABLE_FLT: now also U8.1 (PE2); no longer U8.67 (PE7)
- net TURNTABLE_SW: now also U8.154 (PG10); no longer U8.162 (PB3)
- net at D10.2 (A): now also U8.147 (PD4); no longer U8.155 (PG11)
- net at U8.146 (PD3): now also D11.2 (A)
- net at U8.148 (PD5): now also D9.2 (A)
- net at U8.150 (PD7): now also D8.2 (A)
- net BL_EN: now reaches U8.86 (PB13)
- net BL_DISC: now reaches U8.88 (PB15)
- no-connect marks 44 -> 42
Other:
- note added: "TIM4CH1"
- note added: "TIM4CH2"
- note added: "TIM4CH3"
- note added: "TIM4CH4"
- note removed: "Timer 4 Channel 1"
- note removed: "Timer 4 Channel 2"
- note removed: "Timer 4 Channel 3"
- note removed: "Timer 4 Channel 4"
- moved on the sheet: D10, D11, D8, D9, J4, R25, R26, R27, R28

Commit message: all part numbers
may need revisions
Parts:
- C28, C29: MANUFACTURER (none) -> Murata; Manufacturer_Part_Number (none) -> GRM1885C1H150JA01J
- C30, C32, C35, C37, C38, C40, C41, C42, C44, C45, C46, C47, C49, C51, C52, C53, C54, C55, C56, C57: MANUFACTURER (none) -> Murata; Manufacturer_Part_Number (none) -> GCJ188R71H104KA12D
- C31, C36, C48: MANUFACTURER (none) -> Murata; Manufacturer_Part_Number (none) -> GRM21BR71E225KE11L
- C33, C34, C39, C50, C59, C60, C61, C62, C63, C64: MANUFACTURER (none) -> Murata; Manufacturer_Part_Number (none) -> GCM21BR71E105KA56L
- C43, C58: MANUFACTURER (none) -> Murata; Manufacturer_Part_Number (none) -> GRM219R61E475MA73D
- D10: MANUFACTURER (none) -> Wurth; Manufacturer_Part_Number (none) -> 150080YS75000
- D11: MANUFACTURER (none) -> Wurth; Manufacturer_Part_Number (none) -> 150080RS75000
- D7: MANUFACTURER (none) -> Diodes Incorporated; Manufacturer_Part_Number (none) -> DESD5V0U1BA-7
- D8: MANUFACTURER (none) -> Wurth; Manufacturer_Part_Number (none) -> 150080BS75000
- D9: MANUFACTURER (none) -> Wurth; Manufacturer_Part_Number (none) -> 150080GS75000
- J12, J13: footprint Connector_PinHeader_2.54mm:PinHeader_1x03_P2.54mm_Vertical -> Connector_Molex:Molex_KK-254_AE-6410-03A_1x03_P2.54mm_Vertical; MANUFACTURER (none) -> Molex; Manufacturer_Part_Number (none) -> 0022232031
- R21, R22, R24: MANUFACTURER (none) -> Yageo; Manufacturer_Part_Number (none) -> RC0805JR-0710KL
- R23, R30, R31: MANUFACTURER (none) -> Yageo; Manufacturer_Part_Number (none) -> RC0805FR-074K7L
- R25: MANUFACTURER (none) -> Yageo; Manufacturer_Part_Number (none) -> RC0805FR-0733RL
- R26, R27, R28: MANUFACTURER (none) -> Yageo; Manufacturer_Part_Number (none) -> RC0805JR-07100RL
- R29: MANUFACTURER (none) -> Yageo; Manufacturer_Part_Number (none) -> RC0805FR-071ML
- R32, R33: MANUFACTURER (none) -> Yageo; Manufacturer_Part_Number (none) -> RC0805JR-075K1L
- TP1: footprint TestPoint:TestPoint_Loop_D2.54mm_Drill1.5mm_Beaded -> TestPoint:TestPoint_Pad_D1.5mm; now left out of the parts list
- TP2, TP3, TP4, TP5: now left out of the parts list

Commit message: Final changes before submission to website
Connections:
- net PG_ADJ: now also U8.36 (PC2_C)
- net PG_5V: now reaches U8.37 (PC3_C)
- no-connect marks 42 -> 40
Other:
- note added: "TIM12CH1"
- note removed: "Timer 12 Channel 1"
Changed lines of the file:
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@@
 		)
 	)
-	(text "Timer 12 Channel 1"
+	(text "TIM12CH1"
 		(exclude_from_sim no)
-		(at 271.78 125.222 0)
+		(at 267.462 124.968 0)
 		(effects
 			(font
@@
 	)
 	(no_connect
-		(at 246.38 140.97)
-	)
-	(no_connect
 		(at 149.86 168.91)
 	)
@@
 	)
 	(no_connect
-		(at 246.38 138.43)
-	)
-	(no_connect
 		(at 149.86 87.63)
 	)
@@
 	(wire
 		(pts
+			(xy 246.38 138.43) (xy 261.62 138.43)
+		)
+		(stroke
+			(width 0)
+			(type default)
+		)
+	)
+	(wire
+		(pts
 			(xy 27.94 182.88) (xy 36.83 182.88)
 		)
@@
 	(wire
 		(pts
-			(xy 340.36 161.29) (xy 354.33 161.29)
+			(xy 337.82 160.02) (xy 351.79 160.02)
 		)
 		(stroke
@@
 	(wire
 		(pts
+			(xy 246.38 140.97) (xy 261.62 140.97)
+		)
+		(stroke
+			(width 0)
+			(type default)
+		)
+	)
+	(wire
+		(pts
 			(xy 246.38 54.61) (xy 261.62 54.61)
 		)
@@
 	(wire
 		(pts
-			(xy 340.36 158.75) (xy 354.33 158.75)
+			(xy 337.82 157.48) (xy 351.79 157.48)
 		)
 		(stroke
@@
 		)
 	)
-	(label "PG_PI"
-		(at 340.36 158.75 0)
+	(label "PG_5V"
+		(at 337.82 157.48 0)
 		(effects
 			(font
@@
 	)
 	(label "PG_ADJ"
-		(at 340.36 161.29 0)
+		(at 337.82 160.02 0)
 		(effects
 			(font
@@
 		)
 	)
+	(label "PG_ADJ"
+		(at 261.62 138.43 180)
+		(effects
+			(font
+				(size 1.27 1.27)
+			)
+			(justify right bottom)
+		)
+	)
 	(label "LCD_B7"
 		(at 375.92 81.28 0)
@@
 		)
 	)
+	(label "PG_5V"
+		(at 261.62 140.97 180)
+		(effects
+			(font
+				(size 1.27 1.27)
+			)
+			(justify right bottom)
+		)
+	)
 	(label "USB_DP"
 		(at 367.03 193.04 0)
@@
 		)
 	)
-	(global_label "PG_PI"
+	(global_label "PG_5V"
 		(shape input)
-		(at 354.33 158.75 0)
+		(at 351.79 157.48 0)
 		(fields_autoplaced yes)
 		(effects
@@
 		)
 		(property "Intersheetrefs" "${INTERSHEET_REFS}"
-			(at 362.6976 158.75 0)
+			(at 360.5809 157.48 0)
 			(effects
 				(font
@@
 	(global_label "PG_ADJ"
 		(shape input)
-		(at 354.33 161.29 0)
+		(at 351.79 160.02 0)
 		(fields_autoplaced yes)
 		(effects
@@
 		)
 		(property "Intersheetrefs" "${INTERSHEET_REFS}"
-			(at 364.149 161.29 0)
+			(at 361.609 160.02 0)
 			(effects
 				(font
